Commit message: Week 5 practice. R2D2 moving in RViz

File: src/my_r2d2/urdf/r2d2.urdf.xacro (robot description, xacro)
@@ -37,4 +37,11 @@
     <xacro:default_inertial mass="10"/>
   </link>
+  <link name="base_footprint">
+  </link>
+    <joint name="base_footprint_joint" type="fixed">
+      <parent link="base_footprint"/>
+      <child link="base_link"/>
+      <origin xyz="0 0 ${wheeldiam+0.1+bodylen/2}" rpy="0 0 0"/>
+    </joint>
   <xacro:macro name="wheel" params="prefix suffix reflect">
     <link name="${prefix}_${suffix}_wheel">

Commit message: Week 6. Camera and marker working in RViz

File: src/my_r2d2/urdf/r2d2.urdf.xacro (robot description, xacro)
@@ -220,4 +220,11 @@
     <origin xyz="${.707*width+0.04} 0 ${.707*width}"/>
   </joint>
+  <link name="eye">
+  </link>
+  <joint name="eyejoint" type="fixed">
+    <parent link="box"/>
+    <child link="eye"/>
+    <origin xyz="0.04 0 0" rpy="1.571 3.14 1.571"/>
+  </joint>
   <gazebo>
     <plugin name="gazebo_ros_control" filename="libgazebo_ros_control.so">
